Commit message: Update world and fix image logic

File: catkin_ws/src/my_robot/urdf/my_robot.xacro (robot description, xacro)
@@ -61,5 +61,5 @@
       <origin xyz="0 0 0" rpy=" 0 0 0"/>
       <geometry>
-        <mesh filename="package://my_robot/meshes/hokuyo.dae" />
+        <mesh filename="$(find my_robot)/meshes/hokuyo.dae" />
       </geometry>
     </visual>

Commit message: update robot

File: catkin_ws/src/my_robot/urdf/my_robot.xacro (robot description, xacro)
@@ -77,4 +77,10 @@
     <parent link="chassis"/>
     <child link="camera" />
+  </joint>
+ <link name="camera_optical"></link>
+  <joint name="camera_optical_joint" type="fixed">
+    <origin xyz="0 0 0" rpy="-1.5707 0 -1.5707"/>
+    <parent link="camera"/>
+    <child link="camera_optical"/>
   </joint>
   <link name='left_wheel'>

Commit message: Save updates

File: catkin_ws/src/my_robot/urdf/my_robot.xacro (robot description, xacro)
@@ -1,4 +1,5 @@
 <?xml version='1.0'?>
 <robot name="my_robot" xmlns:xacro="http://www.ros.org/wiki/xacro">
+	<!-- <xacro:include filename="$(find my_robot)/urdf/my_robot.gazebo" /> -->
   <link name="robot_footprint"></link>
   <joint name="robot_footprint_joint" type="fixed">
@@ -78,10 +79,10 @@
     <child link="camera" />
   </joint>
- <link name="camera_optical"></link>
   <joint name="camera_optical_joint" type="fixed">
     <origin xyz="0 0 0" rpy="-1.5707 0 -1.5707"/>
     <parent link="camera"/>
-    <child link="camera_optical"/>
-  </joint>
+    <child link="camera_link_optical"/>
+  </joint>
+  <link name="camera_link_optical"></link>
   <link name='left_wheel'>
      <inertial>
